File: board/BatteryMonitor.kicad_pcb (KiCad board)
At the start: 2 copper layers, 20 parts, among them J1 Screw_Terminal_01x02, J2 Screw_Terminal_01x02, Q1 IPP80P03P4L-04, Q2 2N7000, Q3 IPP80P03P4L-04, U1 OKI-78SR-5_1.5-W36H-C, U2 INA260

Commit message: Finish layout, first spin
Parts:
- added R6: 330, Resistor_SMD:R_0805_2012Metric_Pad1.15x1.40mm_HandSolder, F.Cu at (151.6, 91.4)
- added R7: 330, Resistor_SMD:R_0805_2012Metric_Pad1.15x1.40mm_HandSolder, F.Cu at (156.2, 101.9)
- added REF**: MountingHole_2.7mm_M2.5, MountingHole:MountingHole_2.7mm_M2.5, F.Cu at (174.5, 82.5)
- added REF**: MountingHole_2.7mm_M2.5, MountingHole:MountingHole_2.7mm_M2.5, F.Cu at (174.5, 100.3)
- added REF**: MountingHole_2.7mm_M2.5, MountingHole:MountingHole_2.7mm_M2.5, F.Cu at (83.6, 82.5)
- added REF**: MountingHole_2.7mm_M2.5, MountingHole:MountingHole_2.7mm_M2.5, F.Cu at (83.6, 100.3)
- Q1, Q3: footprint Package_TO_SOT_THT:TO-220-3_Vertical -> Package_TO_SOT_THT:TO-220-3_Horizontal_TabDown
- R1: value 10k -> 100k
- moved R4 84.9 mm to (132.1, 86.1), turned to 90 degrees
- moved D2 77.5 mm to (118.1, 86.4)
- moved R2 73.7 mm to (129.5, 86.1), turned to 270 degrees
- moved Q2 71.2 mm to (138.4, 85.1), turned to 180 degrees
- moved R3 68.4 mm to (142.2, 86.1), turned to 270 degrees
- moved Q3 68.3 mm to (129.5, 91.4), turned to 270 degrees
- moved J2 67.8 mm to (172.7, 88.9), turned to 270 degrees
- moved R1 62.9 mm to (103.6, 86.4), turned to 90 degrees
- moved U1 62.1 mm to (94.2, 85.1)
- moved Q1 62.1 mm to (106.5, 91.4), turned to 270 degrees
- moved D1 57.4 mm to (114.3, 86.4), turned to 180 degrees
- moved J1 51.9 mm to (85.3, 94.0), turned to 90 degrees
- moved R5 47.7 mm to (156.2, 81.0)
- moved D3 45.1 mm to (154.9, 83.8)
- moved C1 34.1 mm to (163.3, 85.3), turned to 90 degrees
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Connections:
- D4 pad 1: Net-(D3-Pad1) -> Net-(D4-Pad1)
- D5 pad 1: Net-(D3-Pad1) -> Net-(D5-Pad1)
- R5 pad 1: Net-(D3-Pad1) -> GND
- R5 pad 2: GND -> Net-(D3-Pad1)
Routing:
- net +BATT: track 0.00 -> 92.5 mm, vias 0 -> 2
- net /RED: track 0.00 -> 81.4 mm, vias 0 -> 2
- net +3V3: track 0.00 -> 74.8 mm
- net /SCL: track 0.00 -> 30.2 mm
- net /YELLOW: track 0.00 -> 27.0 mm
- net /SDA: track 0.00 -> 26.1 mm
- net /GREEN: track 0.00 -> 21.6 mm, vias 0 -> 1
- net +5V: track 0.00 -> 20.4 mm
- net /ENABLE: track 0.00 -> 12.9 mm
- net GND: track 0.00 -> 11.6 mm, vias 0 -> 10
- net Net-(D2-Pad2): track 0.00 -> 11.0 mm
- net Net-(D1-Pad2): track 0.00 -> 8.87 mm
- net Net-(Q3-Pad2): track 0.00 -> 3.81 mm
- net Net-(Q2-Pad3): track 0.00 -> 3.81 mm
- net Net-(D3-Pad1): track 0.00 -> 3.74 mm
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- added copper zone on F.Cu, net +BATT
- added copper zone on B.Cu, net GND
- added copper zone on F.Cu, net GND
- added copper zone on F.Cu, net Net-(J1-Pad2)
- added copper zone on F.Cu, net Net-(J2-Pad1)
- added copper zone on F.Cu, net Net-(Q3-Pad2)
Other:
- board outline added: 98.6 x 25.4 mm
- board text added: "+"
- board text added: "-"
- board text added: "SaintGimp Battery Monitor v1.0.0"
